Commit message: pickup code

File: code/robots/panda_gripper.urdf (robot description, URDF)
Before this commit: robot panda, 9 links, 8 joints
Joints:
- joint panda_finger_joint1: limit lower=0.0 upper=0.06 effort=20 velocity=0.2 -> lower=0.0 upper=0.04 effort=20 velocity=0.2
- joint panda_finger_joint2: limit lower=0.0 upper=0.06 effort=20 velocity=0.2 -> lower=0.0 upper=0.04 effort=20 velocity=0.2

Commit message: Revert "pickup code"
This reverts commit a69d2551e9168d2430d7475077419a759a129870.

File: code/robots/panda_gripper.urdf (robot description, URDF)
Before this commit: robot panda, 9 links, 8 joints
Joints:
- joint panda_finger_joint1: limit lower=0.0 upper=0.04 effort=20 velocity=0.2 -> lower=0.0 upper=0.06 effort=20 velocity=0.2
- joint panda_finger_joint2: limit lower=0.0 upper=0.04 effort=20 velocity=0.2 -> lower=0.0 upper=0.06 effort=20 velocity=0.2
